File: blinkyboard.kicad_sch (KiCad schematic)
At the start: 20 parts, among them J1 Conn_01x02_Socket, SW1 SW_Push, U1 NE555P, U2 4017

Commit message: Upload updated schematic
Connections:
- net +5V: now also SW1.1
Changed lines of the file:
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@@
+	)
+	(junction
+		(at 190.5 67.31)
+		(diameter 0)
+		(color 0 0 0 0)
 	)
 	(junction
@@
 	(wire
 		(pts
+			(xy 190.5 67.31) (xy 190.5 69.85)
+		)
+		(stroke
+			(width 0)
+			(type default)
+		)
+	)
+	(wire
+		(pts
 			(xy 148.59 105.41) (xy 129.54 105.41)
 		)
@@
 		(pts
 			(xy 207.01 95.25) (xy 207.01 104.14)
+		)
+		(stroke
+			(width 0)
+			(type default)
+		)
+	)
+	(wire
+		(pts
+			(xy 190.5 66.04) (xy 190.5 67.31)
 		)
 		(stroke
@@
 	(symbol
 		(lib_id "power:+5V")
-		(at 190.5 69.85 0)
+		(at 190.5 66.04 0)
 		(unit 1)
 		(exclude_from_sim no)
@@
 		(fields_autoplaced yes)
 		(property "Reference" "#PWR09"
-			(at 190.5 73.66 0)
+			(at 190.5 69.85 0)
 			(effects
 				(font
@@
 		)
 		(property "Value" "+5V"
-			(at 190.5 64.77 0)
+			(at 190.5 60.96 0)
 			(effects
 				(font
@@
 		)
 		(property "Footprint" ""
-			(at 190.5 69.85 0)
+			(at 190.5 66.04 0)
 			(effects
 				(font
@@
 		)
 		(property "Datasheet" ""
-			(at 190.5 69.85 0)
+			(at 190.5 66.04 0)
 			(effects
 				(font
@@
 		)
 		(property "Description" "Power symbol creates a global label with name \"+5V\""
-			(at 190.5 69.85 0)
-			(effects
-				(font
+			(at 190.5 66.04 0)
+			(effects
+				(font

Commit message: Update schematic
Other:
- note added: "PAUSE"

Commit message: Final update for KiCad files.
Connections:
- net +5V: now also J1.1 (Pin_1)
- net GND: now also J1.2 (Pin_2)
Other:
- note added: "1 - POWER PIN"
- note added: "2 - GROUNDING PIN"
Changed lines of the file:
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@@
 	(generator_version "9.0")
 	(paper "A4")
+	(text "1 - POWER PIN"
+		(exclude_from_sim no)
+		(at 139.7 58.42 0)
+		(effects
+			(font
+				(size 1.27 1.27)
+			)
+		)
+	)
+	(text "2 - GROUNDING PIN"
+		(exclude_from_sim no)
+		(at 141.986 68.58 0)
+		(effects
+			(font
+				(size 1.27 1.27)
+			)
+		)
+	)
 	(text "PAUSE"
 		(exclude_from_sim no)
@@
 	)
 	(symbol
+		(lib_id "power:+5V")
+		(at 134.62 62.23 90)
+		(unit 1)
+		(exclude_from_sim no)
+		(in_bom yes)
+		(on_board yes)
+		(dnp no)
+		(fields_autoplaced yes)
+		(property "Reference" "#PWR011"
+			(at 138.43 62.23 0)
+			(effects
+				(font
+					(size 1.27 1.27)
+				)
+				(hide yes)
+			)
+		)
+		(property "Value" "+5V"
+			(at 130.81 62.2299 90)
+			(effects
+				(font
+					(size 1.27 1.27)
+				)
+				(justify left)
+			)
+		)
+		(property "Footprint" ""
+			(at 134.62 62.23 0)
+			(effects
+				(font
+					(size 1.27 1.27)
+				)
+				(hide yes)
+			)
+		)
+		(property "Datasheet" ""
+			(at 134.62 62.23 0)
+			(effects
+				(font
+					(size 1.27 1.27)
+				)
+				(hide yes)
+			)
+		)
+		(property "Description" "Power symbol creates a global label with name \"+5V\""
+			(at 134.62 62.23 0)
+			(effects
+				(font
+					(size 1.27 1.27)
+				)
+				(hide yes)
+			)
+		)
+		(pin "1"
+		)
+		(instances
+			(project ""
+				(path "/3b2e93e2-a2cf-49ab-9c21-692f479897da"
+					(reference "#PWR011")
+					(unit 1)
+				)
+			)
+		)
+	)
+	(symbol
 		(lib_id "power:GND")
 		(at 177.8 85.09 0)
@@
 					(unit 1)
 				)
+			)
+		)
+	)
+	(symbol
+		(lib_id "power:GND")
+		(at 134.62 64.77 270)
+		(unit 1)
+		(exclude_from_sim no)
+		(in_bom yes)
+		(on_board yes)
+		(dnp no)
+		(fields_autoplaced yes)
+		(property "Reference" "#PWR012"
+			(at 128.27 64.77 0)
+			(effects
+				(font
+					(size 1.27 1.27)
+				)
+				(hide yes)
+			)
+		)
+		(property "Value" "GND"
+			(at 130.81 64.7699 90)
+			(effects
+				(font
+					(size 1.27 1.27)
+				)
+				(justify right)
+			)
+		)
+		(property "Footprint" ""
+			(at 134.62 64.77 0)
+			(effects
+				(font
+					(size 1.27 1.27)
+				)
+				(hide yes)
+			)
+		)
+		(property "Datasheet" ""
+			(at 134.62 64.77 0)
+			(effects
+				(font
+					(size 1.27 1.27)
+				)
+				(hide yes)
+			)
+		)
+		(property "Description" "Power symbol creates a global label with name \"GND\" , ground"
+			(at 134.62 64.77 0)
+			(effects
+				(font
+					(size 1.27 1.27)
+				)
+				(hide yes)
+			)
+		)
+		(pin "1"
+		)
+		(instances
+			(project ""
+				(path "/3b2e93e2-a2cf-49ab-9c21-692f479897da"
+					(reference "#PWR012")
+					(unit 1)
+				)
